File: BoardDesign/LabBenchPowerSupply.sch (KiCad schematic (older format))
At the start: 50 parts, among them P1 Digital, P2 Analog, P3 CONN_01X01, P4 CONN_01X01, P5 CONN_01X01, P6 CONN_01X01

Commit message: Modified circuitry to only have one buck converter with an antilatchup driver circuitry
Signed-off-by: bebenlebricolo <benoittarrade@hotmail.fr>
Parts:
- removed C?: CP1, symbol Device:CP1
- removed D?: D_Schottky, symbol Device:D_Schottky
- removed Q? (x2): 2N2222, Package_TO_SOT_THT:TO-39-3, symbol Transistor_BJT:2N2219
- removed R? (x5): 1k, symbol Device:R
- removed R?: 56k, symbol Device:R
- removed U?: IRFZ14PBF, symbol NMOS_TH:IRFZ14PBF
- removed U?: LM7805_TO220, Package_TO_SOT_THT:TO-220-3_Vertical, symbol Regulator_Linear:LM7805_TO220
- added C?: 470µ, symbol Device:CP1
- added D?: D, symbol Device:D
- added J? (x2): Conn_01x02, symbol Connector_Generic:Conn_01x02
- added Q? (x2): BC307, Package_TO_SOT_THT:TO-92_Inline, symbol Transistor_BJT:BC307
- added Q?: 2N2222, Package_TO_SOT_THT:TO-39-3, symbol Transistor_BJT:2N2219
- added R? (x3): 56k, symbol Device:R
- added R? (x4): 1k, symbol Device:R
- R?: value 150k -> 220k
Connections:
- net labels added: 10v_smoothed, 23v_smoothed, Vcc(5v), fan_control, minus_button, mode_button, mosfet_low_side, plus_button, var_select_button
- net labels removed: 12Vsmoothed, BOOST_CONTROL, BUCK_CONTROL, FAN_CONTROL, MEMORY_BUTTON, MINUS_BUTTON, PLUS_BUTTON, VARIABLE_BUTTON, Vcc(4.4V), boost_mosfet
- wire segments 149 -> 152
Other:
- note added: "220 V AC / 2x11.5 serie = 23V AC"
- note added: "23V"
- note added: "External buck converter board 23 -> 5V"
- note added: "Note : usually most of generic power mosfets are tolerant to \n30V between Gate and Source. If so, you can either connect the \n23V smoothed line instead of the 10V one, as a power line to \ncontrol the mosfet."
- note added: "Power MOSFET transistors driver section with \nanti-latch protection (single input which controls\nboth sides of the mosfet driver section)"
- note added: "Power section (Buck converter)"
- note removed: "220 V AC / 12 V AC"
- note removed: "Power MOSFET transistors driver section (minimalist implementation of it)"
- moved on the sheet: C?, D?, L?, Q?, R?, SW?, U?
